Commit message: update urdf, add timeout param, fix bug

File: rm_description/urdf/rm_65.urdf (robot description, URDF)
Before this commit: robot rm_65_description, 7 links, 6 joints
Links:
- link Link1: mass 0.593563443690403 -> 1.51
- link Link2: mass 0.864175046869043 -> 1.653
- link Link3: mass 0.289633681624654 -> 0.726
- link Link4: mass 0.239419768320061 -> 0.671
- link Link5: mass 0.218799761431678 -> 0.647
- link Link6: mass 0.0649018034311231 -> 0.104
- link base_link: mass 0.841070778135659 -> 1.862

File: rm_description/urdf/rm_65_6f.urdf (robot description, URDF)
Before this commit: robot rm_65_6f_description, 7 links, 6 joints
Links:
- link Link1: mass 0.59356 -> 1.51
- link Link2: mass 0.86418 -> 1.653
- link Link3: mass 0.28963 -> 0.726
- link Link4: mass 0.23941 -> 0.671
- link Link5: mass 0.21879 -> 0.647
- link Link6: mass 0.14433 -> 0.14434
- link base_link: mass 0.84105 -> 1.862

File: rm_description/urdf/rm_65_6fb.urdf (robot description, URDF)
Before this commit: robot RM65-6F, 7 links, 6 joints
Links:
- link Link1: mass 0.593542243994357 -> 1.51
- link Link2: mass 0.86417584142394 -> 1.653
- link Link3: mass 0.289643824525119 -> 0.726
- link Link4: mass 0.239430992940448 -> 0.671
- link Link5: mass 0.21879527056675 -> 0.647
- link Link6: mass 3.04449097371379 -> 0.14434
- link base_link: mass 0.838885281114303 -> 1.862

File: rm_description/urdf/rm_75.urdf (robot description, URDF)
Before this commit: robot rm_75_description, 8 links, 7 joints
Links:
- link Link1: mass 0.593563458735581 -> 1.574
- link Link2: mass 0.432849770310974 -> 1.217
- link Link3: mass 0.431325495678459 -> 1.11
- link Link4: mass 0.289633681619295 -> 0.685
- link Link5: mass 0.239419768320061 -> 0.619
- link Link6: mass 0.218799761431682 -> 0.602
- link Link7: mass 0.0649018034311231 -> 0.107
- link base_link: mass 0.841071174772543 -> 1.862

File: rm_description/urdf/rm_75_6f.urdf (robot description, URDF)
Before this commit: robot rm_75_6f_description, 8 links, 7 joints
Links:
- link Link1: mass 0.59356 -> 1.574
- link Link2: mass 0.43285 -> 1.217
- link Link3: mass 0.43132 -> 1.11
- link Link4: mass 0.28963 -> 0.685
- link Link5: mass 0.23941 -> 0.619
- link Link6: mass 0.21879 -> 0.602
- link Link7: mass 0.14433 -> 0.144
- link base_link: mass 0.84105 -> 1.862

File: rm_description/urdf/rm_75_6fb.urdf (robot description, URDF)
Before this commit: robot RM75-6F, 8 links, 7 joints
Links:
- link Link7: mass 3.04449097310784 -> 0.144
- link Link_1: mass 0.593542243994357 -> 1.574
- link Link_2: mass 0.432849544766671 -> 1.217
- link Link_3: mass 0.431326296657269 -> 1.11
- link Link_4: mass 0.289643824188822 -> 0.685
- link Link_5: mass 0.239430992940448 -> 0.619
- link Link_6: mass 0.21879527056675 -> 0.602
- link base_link: mass 0.838885280844642 -> 1.862

File: rm_description/urdf/rm_eco63.urdf (robot description, URDF)
Before this commit: robot rm_eco63, 8 links, 7 joints
Links:
- link Link1: mass 0.656374618338142 -> 1.6026
- link Link2: mass 5.26262523683375 -> 2.8169
- link Link3: mass 1.3509329667983 -> 2.6857
- link Link4: mass 0.733001235394853 -> 0.625
- link Link5: mass 0.911747774463918 -> 0.6743
- link Link6: mass 0.065035417997418 -> 0.107
- link base_link: mass 8.97974481667473 -> 1

File: rm_description/urdf/rm_eco63_6fb.urdf (robot description, URDF)
Before this commit: robot ECO63-6FB-URDF, 7 links, 6 joints
Links:
- link Link1: mass 0.656374618338142 -> 1.6026
- link Link2: mass 5.26262523683375 -> 2.8169
- link Link3: mass 1.3509329667983 -> 2.6857
- link Link4: mass 0.733001235394853 -> 0.625
- link Link5: mass 0.911747774463918 -> 0.6743
- link Link6: mass 0.151764173288042 -> 0.248
- link base_link: mass 9.06647326360739 -> 1

File: rm_description/urdf/rm_eco65.urdf (robot description, URDF)
Before this commit: robot rm_eco65_description, 7 links, 6 joints
Links:
- link Link1: mass 0.74247 -> 1.507
- link Link2: mass 1.3502 -> 2.0227
- link Link3: mass 1.0422 -> 1.8858
- link Link4: mass 0.27383 -> 0.57
- link Link5: mass 0.27794 -> 0.641
- link Link6: mass 0.033025 -> 0.0857
- link baselink: mass 0.61127 -> 2

File: rm_description/urdf/rm_eco65_6f.urdf (robot description, URDF)
Before this commit: robot eco65, 7 links, 6 joints
Links:
- link Link1: mass 0.74252212802658 -> 1.507
- link Link2: mass 1.35020712394805 -> 2.0227
- link Link3: mass 1.0422213139163 -> 1.8858
- link Link4: mass 0.273792481713346 -> 0.57
- link Link5: mass 0.27793758472494 -> 0.641
- link Link6: mass 0.14611108984048 -> 0.0857
- link baselink: mass 0.61127 -> 2

File: rm_description/urdf/rm_eco65_6fb.urdf (robot description, URDF)
Before this commit: robot 0000-eco65_URDF(2), 7 links, 6 joints
Links:
- link base_link: mass 1.6314377241954 -> 2
- link link1: mass 1.76684172446222 -> 1.507
- link link2: mass 3.5404490739212 -> 2.0227
- link link3: mass 2.66024465891583 -> 1.8858
- link link4: mass 0.733002748293818 -> 0.57
- link link5: mass 0.911746755408486 -> 0.641
- link link6: mass 0.305602477849543 -> 0.0857

File: rm_description/urdf/rm_rx75-6fb.urdf.xacro (robot description, xacro)
@@ -447,5 +447,5 @@
     <visual>
       <origin
-        xyz="0 -0.119000004117148 0"
+        xyz="0 -0.0962 0"
         rpy="1.57079632679489 0 0" />
       <geometry>
@@ -461,5 +461,5 @@
     <collision>
       <origin
-        xyz="0 -0.119000004117148 0"
+        xyz="0 -0.0962 0"
         rpy="1.57079632679489 0 0" />
       <geometry>
@@ -493,5 +493,5 @@
     type="fixed">
     <origin
-      xyz="0 -0.119000004117148 0"
+      xyz="0 -0.0962 0"
       rpy="1.57079632679489 0 0" />
     <parent
@@ -930,5 +930,5 @@
     <visual>
       <origin
-        xyz="0 0.119000004117148 0"
+        xyz="0 0.0962 0"
         rpy="-1.5707963267949 0 0" />
       <geometry>
@@ -944,5 +944,5 @@
     <collision>
       <origin
-        xyz="0 0.119000004117148 0"
+        xyz="0 0.0962 0"
         rpy="-1.5707963267949 0 0" />
       <geometry>
@@ -975,5 +975,5 @@
     type="fixed">
     <origin
-      xyz="0 0.119000004117148 0"
+      xyz="0 0.0962 0"
       rpy="-1.5707963267949 0 0" />
     <parent

File: rm_description/urdf/rm_rx75l-6fb.urdf (robot description, URDF)
Before this commit: robot RXL-6FB, 9 links, 8 joints
Joints:
- joint J8: origin xyz=0 -0.119000004117148 0 rpy=1.57079632679489 0 0 -> xyz=0 -0.0962 0 rpy=1.57079632679489 0 0

File: rm_description/urdf/rm_rx75r-6fb.urdf (robot description, URDF)
Before this commit: robot RXR-6FB, 9 links, 8 joints
Joints:
- joint J8: origin xyz=0 0.119000004117148 0 rpy=-1.5707963267949 0 0 -> xyz=0 0.0962 0 rpy=-1.5707963267949 0 0

File: rm_description/urdf/rml_63.urdf (robot description, URDF)
Before this commit: robot rml_63_description, 7 links, 6 joints
Links:
- link base_link: mass 0.66248 -> 1.862
- link link1: mass 1.7668 -> 1.837
- link link2: mass 4.3415 -> 2.006
- link link3: mass 1.7286 -> 1.961
- link link4: mass 2.4734 -> 1.201
- link link5: mass 0.93162 -> 1.026
- link link6: mass 0.065037 -> 0.107

File: rm_description/urdf/rml_63_6f.urdf (robot description, URDF)
Before this commit: robot rm_63_6f_description, 7 links, 6 joints
Links:
- link Link1: mass 0.92308 -> 1.837
- link Link2: mass 1.5577 -> 2.006
- link Link3: mass 0.71556 -> 1.961
- link Link4: mass 0.69692 -> 1.201
- link Link5: mass 0.3567 -> 1.026
- link Link6: mass 0.14814 -> 0.248
- link base_link: mass 0.66248 -> 1.862

File: rm_description/urdf/rml_63_6fb.urdf (robot description, URDF)
Before this commit: robot RML-63-6F, 7 links, 6 joints
Links:
- link Link_1: mass 1.7668 -> 1.837
- link Link_2: mass 4.3415 -> 2.006
- link Link_3: mass 1.7286 -> 1.961
- link Link_4: mass 2.4734 -> 1.201
- link Link_5: mass 0.93162 -> 1.026
- link Link_6: mass 0.3056 -> 0.248
- link base_link: mass 1.6314 -> 1.862
