Commit message: fix: correct robot joint frames in URDF files

File: rm_description/urdf/rm_75_6fb.urdf (robot description, URDF)
Before this commit: robot RM75-6F, 8 links, 7 joints
Joints:
- joint joint7: origin xyz=0 -0.1613 0 rpy=1.5708 0 0 -> xyz=0 0 0.1612 rpy=0 0 0
- joint joint_1: axis 0 0 -1 -> 0 -1 0; origin xyz=0 0 0.2405 rpy=0 0 0 -> xyz=0 0 0.2405 rpy=-1.5708 0 0
- joint joint_2: axis 0 0 1 -> 0 1 0; origin xyz=0 0 0 rpy=1.5708 -1.5708 0 -> xyz=0 0 0 rpy=1.5708 0 0
- joint joint_3: axis 0 0 -1 -> 0 -1 0; origin xyz=0.256 0 0 rpy=-1.5708 0 -1.5708 -> xyz=0 0 0.256 rpy=-1.5708 0 0
- joint joint_4: axis 0 0 1 -> 0 1 0; origin xyz=0 0 0 rpy=-1.5708 0 -3.1416 -> xyz=0 0 0 rpy=1.5708 0 0
- joint joint_5: axis 0 0 -1 -> 0 -1 0; origin xyz=0 -0.21 0 rpy=1.5708 0 0 -> xyz=0 0 0.21 rpy=-1.5708 0 0
- joint joint_6: axis 0 0 1 -> 0 1 0; origin xyz=0 0 0 rpy=-1.5708 0 0 -> xyz=0 0 0 rpy=1.5708 0 0

File: rm_description/urdf/rm_eco65_6fb.urdf (robot description, URDF)
Before this commit: robot 0000-eco65_URDF(2), 7 links, 6 joints
Joints:
- joint joint2: origin xyz=-0.086 0 0 rpy=-1.5708 -1.5708 0 -> xyz=-0.086 0 0 rpy=1.5708 0 0
- joint joint3: origin xyz=0.26 0 0 rpy=0 0 0 -> xyz=0 0.26 0 rpy=3.1416 0 1.5708

File: rm_description/urdf/rml_63_6fb.urdf (robot description, URDF)
Before this commit: robot RML-63-6F, 7 links, 6 joints
Joints:
- joint joint_1: origin xyz=0 0 0.1625 rpy=0 0 0 -> xyz=0 0 0.172 rpy=0 0 0

File: rm_description/urdf/rml_63_6fb_description.urdf.xacro (robot description, xacro)
@@ -138,5 +138,5 @@
     type="revolute">
     <origin
-      xyz="0 0 0.1625"
+      xyz="0 0 0.172"
       rpy="0 0 0" />
     <parent
