Commit message: fix: 修正 ECO65 模型网格路径

File: rm_description/urdf/rm_eco65.urdf (robot description, URDF)
Before this commit: robot rm_eco65_description, 7 links, 6 joints
Links:
- link Link1: geometry collision mesh filename=package://rm_description/meshes/rm_eco65_arm/Link_1.STL; visual mesh filename=package://rm_description/meshes/rm_eco65_arm/Link_1.STL
- link Link2: geometry collision mesh filename=package://rm_description/meshes/rm_eco65_arm/Link_2.STL; visual mesh filename=package://rm_description/meshes/rm_eco65_arm/Link_2.STL
- link Link3: geometry collision mesh filename=package://rm_description/meshes/rm_eco65_arm/Link_3.STL; visual mesh filename=package://rm_description/meshes/rm_eco65_arm/Link_3.STL
- link Link4: geometry collision mesh filename=package://rm_description/meshes/rm_eco65_arm/Link_4.STL; visual mesh filename=package://rm_description/meshes/rm_eco65_arm/Link_4.STL
- link Link5: geometry collision mesh filename=package://rm_description/meshes/rm_eco65_arm/Link_5.STL; visual mesh filename=package://rm_description/meshes/rm_eco65_arm/Link_5.STL

File: rm_description/urdf/rm_eco65.urdf.xacro (robot description, xacro)
@@ -67,5 +67,5 @@
       <geometry>
         <mesh
-          filename="package://rm_description/meshes/rm_eco65_arm/Link1.STL" />
+          filename="package://rm_description/meshes/rm_eco65_arm/Link_1.STL" />
       </geometry>
       <material
@@ -81,5 +81,5 @@
       <geometry>
         <mesh
-          filename="package://rm_description/meshes/rm_eco65_arm/Link1.STL" />
+          filename="package://rm_description/meshes/rm_eco65_arm/Link_1.STL" />
       </geometry>
     </collision>
@@ -125,5 +125,5 @@
       <geometry>
         <mesh
-          filename="package://rm_description/meshes/rm_eco65_arm/Link2.STL" />
+          filename="package://rm_description/meshes/rm_eco65_arm/Link_2.STL" />
       </geometry>
       <material
@@ -139,5 +139,5 @@
       <geometry>
         <mesh
-          filename="package://rm_description/meshes/rm_eco65_arm/Link2.STL" />
+          filename="package://rm_description/meshes/rm_eco65_arm/Link_2.STL" />
       </geometry>
     </collision>
@@ -183,5 +183,5 @@
       <geometry>
         <mesh
-          filename="package://rm_description/meshes/rm_eco65_arm/Link3.STL" />
+          filename="package://rm_description/meshes/rm_eco65_arm/Link_3.STL" />
       </geometry>
       <material
@@ -197,5 +197,5 @@
       <geometry>
         <mesh
-          filename="package://rm_description/meshes/rm_eco65_arm/Link3.STL" />
+          filename="package://rm_description/meshes/rm_eco65_arm/Link_3.STL" />
       </geometry>
     </collision>
@@ -241,5 +241,5 @@
       <geometry>
         <mesh
-          filename="package://rm_description/meshes/rm_eco65_arm/Link4.STL" />
+          filename="package://rm_description/meshes/rm_eco65_arm/Link_4.STL" />
       </geometry>
       <material
@@ -255,5 +255,5 @@
       <geometry>
         <mesh
-          filename="package://rm_description/meshes/rm_eco65_arm/Link4.STL" />
+          filename="package://rm_description/meshes/rm_eco65_arm/Link_4.STL" />
       </geometry>
     </collision>
@@ -299,5 +299,5 @@
       <geometry>
         <mesh
-          filename="package://rm_description/meshes/rm_eco65_arm/Link5.STL" />
+          filename="package://rm_description/meshes/rm_eco65_arm/Link_5.STL" />
       </geometry>
       <material
@@ -313,5 +313,5 @@
       <geometry>
         <mesh
-          filename="package://rm_description/meshes/rm_eco65_arm/Link5.STL" />
+          filename="package://rm_description/meshes/rm_eco65_arm/Link_5.STL" />
       </geometry>
     </collision>
@@ -478,5 +478,5 @@
             <geometry>
                 <mesh
-                filename="package://rm_description/meshes/rm_eco65_arm/Link6_6fb.STL" />
+                filename="package://rm_description/meshes/rm_eco65_arm/Link_6fb.STL" />
             </geometry>
             <material
@@ -492,5 +492,5 @@
             <geometry>
                 <mesh
-                filename="package://rm_description/meshes/rm_eco65_arm/Link6_6fb.STL" />
+                filename="package://rm_description/meshes/rm_eco65_arm/Link_6fb.STL" />
             </geometry>
             </collision>

File: rm_description/urdf/rm_eco65_6f.urdf (robot description, URDF)
Before this commit: robot eco65, 7 links, 6 joints
Links:
- link Link1: geometry collision mesh filename=package://rm_description/meshes/rm_eco65_arm/Link_1.STL; visual mesh filename=package://rm_description/meshes/rm_eco65_arm/Link_1.STL
- link Link2: geometry collision mesh filename=package://rm_description/meshes/rm_eco65_arm/Link_2.STL; visual mesh filename=package://rm_description/meshes/rm_eco65_arm/Link_2.STL
- link Link3: geometry collision mesh filename=package://rm_description/meshes/rm_eco65_arm/Link_3.STL; visual mesh filename=package://rm_description/meshes/rm_eco65_arm/Link_3.STL
- link Link4: geometry collision mesh filename=package://rm_description/meshes/rm_eco65_arm/Link_4.STL; visual mesh filename=package://rm_description/meshes/rm_eco65_arm/Link_4.STL
- link Link5: geometry collision mesh filename=package://rm_description/meshes/rm_eco65_arm/Link_5.STL; visual mesh filename=package://rm_description/meshes/rm_eco65_arm/Link_5.STL

File: rm_description/urdf/rm_eco65_6fb.urdf (robot description, URDF)
Before this commit: robot 0000-eco65_URDF(2), 7 links, 6 joints
Links:
- link link1: geometry collision mesh filename=package://rm_description/meshes/rm_eco65_arm/Link_1.STL; visual mesh filename=package://rm_description/meshes/rm_eco65_arm/Link_1.STL
- link link2: geometry collision mesh filename=package://rm_description/meshes/rm_eco65_arm/Link_2.STL; visual mesh filename=package://rm_description/meshes/rm_eco65_arm/Link_2.STL
- link link3: geometry collision mesh filename=package://rm_description/meshes/rm_eco65_arm/Link_3.STL; visual mesh filename=package://rm_description/meshes/rm_eco65_arm/Link_3.STL
- link link4: geometry collision mesh filename=package://rm_description/meshes/rm_eco65_arm/Link_4.STL; visual mesh filename=package://rm_description/meshes/rm_eco65_arm/Link_4.STL
- link link5: geometry collision mesh filename=package://rm_description/meshes/rm_eco65_arm/Link_5.STL; visual mesh filename=package://rm_description/meshes/rm_eco65_arm/Link_5.STL
- link link6: geometry collision mesh filename=package://rm_description/meshes/rm_eco65_arm/Link_6fb.STL; visual mesh filename=package://rm_description/meshes/rm_eco65_arm/Link_6fb.STL

File: rm_description/urdf/rm_eco65_gazebo.urdf (robot description, URDF)
Before this commit: robot rm_eco65_description, 7 links, 6 joints
Links:
- link Link1: geometry collision mesh filename=file://$(find rm_description)/meshes/rm_eco65_arm/Link_1.STL; visual mesh filename=file://$(find rm_description)/meshes/rm_eco65_arm/Link_1.STL
- link Link2: geometry collision mesh filename=file://$(find rm_description)/meshes/rm_eco65_arm/Link_2.STL; visual mesh filename=file://$(find rm_description)/meshes/rm_eco65_arm/Link_2.STL
- link Link3: geometry collision mesh filename=file://$(find rm_description)/meshes/rm_eco65_arm/Link_3.STL; visual mesh filename=file://$(find rm_description)/meshes/rm_eco65_arm/Link_3.STL
- link Link4: geometry collision mesh filename=file://$(find rm_description)/meshes/rm_eco65_arm/Link_4.STL; visual mesh filename=file://$(find rm_description)/meshes/rm_eco65_arm/Link_4.STL
- link Link5: geometry collision mesh filename=file://$(find rm_description)/meshes/rm_eco65_arm/Link_5.STL; visual mesh filename=file://$(find rm_description)/meshes/rm_eco65_arm/Link_5.STL

File: rm_description/urdf/rm_eco65_gazebo.urdf.xacro (robot description, xacro)
@@ -67,5 +67,5 @@
       <geometry>
         <mesh
-          filename="file://$(find rm_description)/meshes/rm_eco65_arm/Link1.STL" />
+          filename="file://$(find rm_description)/meshes/rm_eco65_arm/Link_1.STL" />
       </geometry>
       <material
@@ -81,5 +81,5 @@
       <geometry>
         <mesh
-          filename="file://$(find rm_description)/meshes/rm_eco65_arm/Link1.STL" />
+          filename="file://$(find rm_description)/meshes/rm_eco65_arm/Link_1.STL" />
       </geometry>
     </collision>
@@ -125,5 +125,5 @@
       <geometry>
         <mesh
-          filename="file://$(find rm_description)/meshes/rm_eco65_arm/Link2.STL" />
+          filename="file://$(find rm_description)/meshes/rm_eco65_arm/Link_2.STL" />
       </geometry>
       <material
@@ -139,5 +139,5 @@
       <geometry>
         <mesh
-          filename="file://$(find rm_description)/meshes/rm_eco65_arm/Link2.STL" />
+          filename="file://$(find rm_description)/meshes/rm_eco65_arm/Link_2.STL" />
       </geometry>
     </collision>
@@ -183,5 +183,5 @@
       <geometry>
         <mesh
-          filename="file://$(find rm_description)/meshes/rm_eco65_arm/Link3.STL" />
+          filename="file://$(find rm_description)/meshes/rm_eco65_arm/Link_3.STL" />
       </geometry>
       <material
@@ -197,5 +197,5 @@
       <geometry>
         <mesh
-          filename="file://$(find rm_description)/meshes/rm_eco65_arm/Link3.STL" />
+          filename="file://$(find rm_description)/meshes/rm_eco65_arm/Link_3.STL" />
       </geometry>
     </collision>
@@ -241,5 +241,5 @@
       <geometry>
         <mesh
-          filename="file://$(find rm_description)/meshes/rm_eco65_arm/Link4.STL" />
+          filename="file://$(find rm_description)/meshes/rm_eco65_arm/Link_4.STL" />
       </geometry>
       <material
@@ -255,5 +255,5 @@
       <geometry>
         <mesh
-          filename="file://$(find rm_description)/meshes/rm_eco65_arm/Link4.STL" />
+          filename="file://$(find rm_description)/meshes/rm_eco65_arm/Link_4.STL" />
       </geometry>
     </collision>
@@ -299,5 +299,5 @@
       <geometry>
         <mesh
-          filename="file://$(find rm_description)/meshes/rm_eco65_arm/Link5.STL" />
+          filename="file://$(find rm_description)/meshes/rm_eco65_arm/Link_5.STL" />
       </geometry>
       <material
@@ -313,5 +313,5 @@
       <geometry>
         <mesh
-          filename="file://$(find rm_description)/meshes/rm_eco65_arm/Link5.STL" />
+          filename="file://$(find rm_description)/meshes/rm_eco65_arm/Link_5.STL" />
       </geometry>
     </collision>
@@ -478,5 +478,5 @@
             <geometry>
                 <mesh
-                filename="file://$(find rm_description)/meshes/rm_eco65_arm/Link6_6fb.STL" />
+                filename="file://$(find rm_description)/meshes/rm_eco65_arm/Link_6fb.STL" />
             </geometry>
             <material
@@ -492,5 +492,5 @@
             <geometry>
                 <mesh
-                filename="file://$(find rm_description)/meshes/rm_eco65_arm/Link6_6fb.STL" />
+                filename="file://$(find rm_description)/meshes/rm_eco65_arm/Link_6fb.STL" />
             </geometry>
             </collision>
