Commit message: feat: 改用 DAE 模型并适配 RViz2 和 Gazebo

File: rm_description/urdf/imported/65_6f.urdf.xacro (robot description, xacro)
@@ -16,5 +16,5 @@
       <origin xyz="0 0 0" rpy="0 0 0" />
       <geometry>
-        <mesh filename="package://rm_description/meshes/glb/base/base_v1.0.glb" />
+        <mesh filename="package://rm_description/meshes/dae/base/base_v1.0.dae" />
       </geometry>
     </visual>
@@ -35,5 +35,5 @@
       <origin xyz="0 0 0" rpy="0 0 0" />
       <geometry>
-        <mesh filename="package://rm_description/meshes/glb/rm65/link_1.glb" />
+        <mesh filename="package://rm_description/meshes/dae/rm65/link_1.dae" />
       </geometry>
     </visual>
@@ -61,5 +61,5 @@
       <origin xyz="0 0 0" rpy="0 0 0" />
       <geometry>
-        <mesh filename="package://rm_description/meshes/glb/rm65/link_2.glb" />
+        <mesh filename="package://rm_description/meshes/dae/rm65/link_2.dae" />
       </geometry>
     </visual>
@@ -87,5 +87,5 @@
       <origin xyz="0 0 0" rpy="0 0 0" />
       <geometry>
-        <mesh filename="package://rm_description/meshes/glb/rm65/link_3.glb" />
+        <mesh filename="package://rm_description/meshes/dae/rm65/link_3.dae" />
       </geometry>
     </visual>
@@ -113,5 +113,5 @@
       <origin xyz="0 0 0" rpy="0 0 0" />
       <geometry>
-        <mesh filename="package://rm_description/meshes/glb/rm65/link_4.glb" />
+        <mesh filename="package://rm_description/meshes/dae/rm65/link_4.dae" />
       </geometry>
     </visual>
@@ -139,5 +139,5 @@
       <origin xyz="0 0 0" rpy="0 0 0" />
       <geometry>
-        <mesh filename="package://rm_description/meshes/glb/rm65/link_5.glb" />
+        <mesh filename="package://rm_description/meshes/dae/rm65/link_5.dae" />
       </geometry>
     </visual>
@@ -165,5 +165,5 @@
       <origin xyz="0 0 0" rpy="0 0 0" />
       <geometry>
-        <mesh filename="package://rm_description/meshes/glb/rm65/link_6_f.glb" />
+        <mesh filename="package://rm_description/meshes/dae/rm65/link_6_f.dae" />
       </geometry>
     </visual>

File: rm_description/urdf/imported/65_6fb.urdf.xacro (robot description, xacro)
@@ -16,5 +16,5 @@
       <origin xyz="0 0 0" rpy="0 0 0" />
       <geometry>
-        <mesh filename="package://rm_description/meshes/glb/base/base_v1.0.glb" />
+        <mesh filename="package://rm_description/meshes/dae/base/base_v1.0.dae" />
       </geometry>
     </visual>
@@ -35,5 +35,5 @@
       <origin xyz="0 0 0" rpy="0 0 0" />
       <geometry>
-        <mesh filename="package://rm_description/meshes/glb/rm65/link_1.glb" />
+        <mesh filename="package://rm_description/meshes/dae/rm65/link_1.dae" />
       </geometry>
     </visual>
@@ -61,5 +61,5 @@
       <origin xyz="0 0 0" rpy="0 0 0" />
       <geometry>
-        <mesh filename="package://rm_description/meshes/glb/rm65/link_2.glb" />
+        <mesh filename="package://rm_description/meshes/dae/rm65/link_2.dae" />
       </geometry>
     </visual>
@@ -87,5 +87,5 @@
       <origin xyz="0 0 0" rpy="0 0 0" />
       <geometry>
-        <mesh filename="package://rm_description/meshes/glb/rm65/link_3.glb" />
+        <mesh filename="package://rm_description/meshes/dae/rm65/link_3.dae" />
       </geometry>
     </visual>
@@ -113,5 +113,5 @@
       <origin xyz="0 0 0" rpy="0 0 0" />
       <geometry>
-        <mesh filename="package://rm_description/meshes/glb/rm65/link_4.glb" />
+        <mesh filename="package://rm_description/meshes/dae/rm65/link_4.dae" />
       </geometry>
     </visual>
@@ -139,5 +139,5 @@
       <origin xyz="0 0 0" rpy="0 0 0" />
       <geometry>
-        <mesh filename="package://rm_description/meshes/glb/rm65/link_5.glb" />
+        <mesh filename="package://rm_description/meshes/dae/rm65/link_5.dae" />
       </geometry>
     </visual>
@@ -165,5 +165,5 @@
       <origin xyz="0 0 0" rpy="0 0 0" />
       <geometry>
-        <mesh filename="package://rm_description/meshes/glb/rm65/link_6_fb.glb" />
+        <mesh filename="package://rm_description/meshes/dae/rm65/link_6_fb.dae" />
       </geometry>
     </visual>

File: rm_description/urdf/imported/65_standard.urdf.xacro (robot description, xacro)
@@ -16,5 +16,5 @@
       <origin xyz="0 0 0" rpy="0 0 0" />
       <geometry>
-        <mesh filename="package://rm_description/meshes/glb/base/base_v1.0.glb" />
+        <mesh filename="package://rm_description/meshes/dae/base/base_v1.0.dae" />
       </geometry>
     </visual>
@@ -35,5 +35,5 @@
       <origin xyz="0 0 0" rpy="0 0 0" />
       <geometry>
-        <mesh filename="package://rm_description/meshes/glb/rm65/link_1.glb" />
+        <mesh filename="package://rm_description/meshes/dae/rm65/link_1.dae" />
       </geometry>
     </visual>
@@ -61,5 +61,5 @@
       <origin xyz="0 0 0" rpy="0 0 0" />
       <geometry>
-        <mesh filename="package://rm_description/meshes/glb/rm65/link_2.glb" />
+        <mesh filename="package://rm_description/meshes/dae/rm65/link_2.dae" />
       </geometry>
     </visual>
@@ -87,5 +87,5 @@
       <origin xyz="0 0 0" rpy="0 0 0" />
       <geometry>
-        <mesh filename="package://rm_description/meshes/glb/rm65/link_3.glb" />
+        <mesh filename="package://rm_description/meshes/dae/rm65/link_3.dae" />
       </geometry>
     </visual>
@@ -113,5 +113,5 @@
       <origin xyz="0 0 0" rpy="0 0 0" />
       <geometry>
-        <mesh filename="package://rm_description/meshes/glb/rm65/link_4.glb" />
+        <mesh filename="package://rm_description/meshes/dae/rm65/link_4.dae" />
       </geometry>
     </visual>
@@ -139,5 +139,5 @@
       <origin xyz="0 0 0" rpy="0 0 0" />
       <geometry>
-        <mesh filename="package://rm_description/meshes/glb/rm65/link_5.glb" />
+        <mesh filename="package://rm_description/meshes/dae/rm65/link_5.dae" />
       </geometry>
     </visual>
@@ -165,5 +165,5 @@
       <origin xyz="0 0 0" rpy="0 0 0" />
       <geometry>
-        <mesh filename="package://rm_description/meshes/glb/rm65/link_6_bi.glb" />
+        <mesh filename="package://rm_description/meshes/dae/rm65/link_6_bi.dae" />
       </geometry>
     </visual>

File: rm_description/urdf/imported/75_6f.urdf.xacro (robot description, xacro)
@@ -16,5 +16,5 @@
       <origin xyz="0 0 0" rpy="0 0 0" />
       <geometry>
-        <mesh filename="package://rm_description/meshes/glb/base/base_link_75.glb" />
+        <mesh filename="package://rm_description/meshes/dae/base/base_link_75.dae" />
       </geometry>
     </visual>
@@ -35,5 +35,5 @@
       <origin xyz="0 0 0" rpy="1.57079632679 0 0" />
       <geometry>
-        <mesh filename="package://rm_description/meshes/glb/rm75/link_1.glb" />
+        <mesh filename="package://rm_description/meshes/dae/rm75/link_1.dae" />
       </geometry>
     </visual>
@@ -61,5 +61,5 @@
       <origin xyz="0 0 0" rpy="-1.57079632679 0 0" />
       <geometry>
-        <mesh filename="package://rm_description/meshes/glb/rm75/link_2.glb" />
+        <mesh filename="package://rm_description/meshes/dae/rm75/link_2.dae" />
       </geometry>
     </visual>
@@ -87,5 +87,5 @@
       <origin xyz="0 0 0" rpy="1.57079632679 0 0" />
       <geometry>
-        <mesh filename="package://rm_description/meshes/glb/rm75/link_3.glb" />
+        <mesh filename="package://rm_description/meshes/dae/rm75/link_3.dae" />
       </geometry>
     </visual>
@@ -113,5 +113,5 @@
       <origin xyz="0 0 0" rpy="-1.57079632679 0 0" />
       <geometry>
-        <mesh filename="package://rm_description/meshes/glb/rm75/link_4.glb" />
+        <mesh filename="package://rm_description/meshes/dae/rm75/link_4.dae" />
       </geometry>
     </visual>
@@ -139,5 +139,5 @@
       <origin xyz="0 0 0" rpy="1.57079632679 0 0" />
       <geometry>
-        <mesh filename="package://rm_description/meshes/glb/rm75/link_5.glb" />
+        <mesh filename="package://rm_description/meshes/dae/rm75/link_5.dae" />
       </geometry>
     </visual>
@@ -165,5 +165,5 @@
       <origin xyz="0 0 0" rpy="-1.57079632679 0 0" />
       <geometry>
-        <mesh filename="package://rm_description/meshes/glb/rm75/link_6.glb" />
+        <mesh filename="package://rm_description/meshes/dae/rm75/link_6.dae" />
       </geometry>
     </visual>
@@ -191,5 +191,5 @@
       <origin xyz="0 0 0" rpy="0 0 0" />
       <geometry>
-        <mesh filename="package://rm_description/meshes/glb/rm75/link_7_fi.glb" />
+        <mesh filename="package://rm_description/meshes/dae/rm75/link_7_fi.dae" />
       </geometry>
     </visual>

File: rm_description/urdf/imported/75_6fb.urdf.xacro (robot description, xacro)
@@ -16,5 +16,5 @@
       <origin xyz="0 0 0" rpy="0 0 0" />
       <geometry>
-        <mesh filename="package://rm_description/meshes/glb/base/base_link_75.glb" />
+        <mesh filename="package://rm_description/meshes/dae/base/base_link_75.dae" />
       </geometry>
     </visual>
@@ -35,5 +35,5 @@
       <origin xyz="0 0 0" rpy="1.57079632679 0 0" />
       <geometry>
-        <mesh filename="package://rm_description/meshes/glb/rm75/link_1.glb" />
+        <mesh filename="package://rm_description/meshes/dae/rm75/link_1.dae" />
       </geometry>
     </visual>
@@ -61,5 +61,5 @@
       <origin xyz="0 0 0" rpy="-1.57079632679 0 0" />
       <geometry>
-        <mesh filename="package://rm_description/meshes/glb/rm75/link_2.glb" />
+        <mesh filename="package://rm_description/meshes/dae/rm75/link_2.dae" />
       </geometry>
     </visual>
@@ -87,5 +87,5 @@
       <origin xyz="0 0 0" rpy="1.57079632679 0 0" />
       <geometry>
-        <mesh filename="package://rm_description/meshes/glb/rm75/link_3.glb" />
+        <mesh filename="package://rm_description/meshes/dae/rm75/link_3.dae" />
       </geometry>
     </visual>
@@ -113,5 +113,5 @@
       <origin xyz="0 0 0" rpy="-1.57079632679 0 0" />
       <geometry>
-        <mesh filename="package://rm_description/meshes/glb/rm75/link_4.glb" />
+        <mesh filename="package://rm_description/meshes/dae/rm75/link_4.dae" />
       </geometry>
     </visual>
@@ -139,5 +139,5 @@
       <origin xyz="0 0 0" rpy="1.57079632679 0 0" />
       <geometry>
-        <mesh filename="package://rm_description/meshes/glb/rm75/link_5.glb" />
+        <mesh filename="package://rm_description/meshes/dae/rm75/link_5.dae" />
       </geometry>
     </visual>
@@ -165,5 +165,5 @@
       <origin xyz="0 0 0" rpy="-1.57079632679 0 0" />
       <geometry>
-        <mesh filename="package://rm_description/meshes/glb/rm75/link_6.glb" />
+        <mesh filename="package://rm_description/meshes/dae/rm75/link_6.dae" />
       </geometry>
     </visual>
@@ -191,5 +191,5 @@
       <origin xyz="0 0 0" rpy="0 0 0" />
       <geometry>
-        <mesh filename="package://rm_description/meshes/glb/rm75/link_7_fb.glb" />
+        <mesh filename="package://rm_description/meshes/dae/rm75/link_7_fb.dae" />
       </geometry>
     </visual>

File: rm_description/urdf/imported/75_standard.urdf.xacro (robot description, xacro)
@@ -16,5 +16,5 @@
       <origin xyz="0 0 0" rpy="0 0 0" />
       <geometry>
-        <mesh filename="package://rm_description/meshes/glb/base/base_link_75.glb" />
+        <mesh filename="package://rm_description/meshes/dae/base/base_link_75.dae" />
       </geometry>
     </visual>
@@ -35,5 +35,5 @@
       <origin xyz="0 0 0" rpy="1.57079632679 0 0" />
       <geometry>
-        <mesh filename="package://rm_description/meshes/glb/rm75/link_1.glb" />
+        <mesh filename="package://rm_description/meshes/dae/rm75/link_1.dae" />
       </geometry>
     </visual>
@@ -61,5 +61,5 @@
       <origin xyz="0 0 0" rpy="-1.57079632679 0 0" />
       <geometry>
-        <mesh filename="package://rm_description/meshes/glb/rm75/link_2.glb" />
+        <mesh filename="package://rm_description/meshes/dae/rm75/link_2.dae" />
       </geometry>
     </visual>
@@ -87,5 +87,5 @@
       <origin xyz="0 0 0" rpy="1.57079632679 0 0" />
       <geometry>
-        <mesh filename="package://rm_description/meshes/glb/rm75/link_3.glb" />
+        <mesh filename="package://rm_description/meshes/dae/rm75/link_3.dae" />
       </geometry>
     </visual>
@@ -113,5 +113,5 @@
       <origin xyz="0 0 0" rpy="-1.57079632679 0 0" />
       <geometry>
-        <mesh filename="package://rm_description/meshes/glb/rm75/link_4.glb" />
+        <mesh filename="package://rm_description/meshes/dae/rm75/link_4.dae" />
       </geometry>
     </visual>
@@ -139,5 +139,5 @@
       <origin xyz="0 0 0" rpy="1.57079632679 0 0" />
       <geometry>
-        <mesh filename="package://rm_description/meshes/glb/rm75/link_5.glb" />
+        <mesh filename="package://rm_description/meshes/dae/rm75/link_5.dae" />
       </geometry>
     </visual>
@@ -165,5 +165,5 @@
       <origin xyz="0 0 0" rpy="-1.57079632679 0 0" />
       <geometry>
-        <mesh filename="package://rm_description/meshes/glb/rm75/link_6.glb" />
+        <mesh filename="package://rm_description/meshes/dae/rm75/link_6.dae" />
       </geometry>
     </visual>
@@ -191,5 +191,5 @@
       <origin xyz="0 0 0" rpy="0 0 0" />
       <geometry>
-        <mesh filename="package://rm_description/meshes/glb/rm75/link_7.glb" />
+        <mesh filename="package://rm_description/meshes/dae/rm75/link_7.dae" />
       </geometry>
     </visual>

File: rm_description/urdf/imported/eco62_standard.urdf.xacro (robot description, xacro)
@@ -22,5 +22,5 @@
       <origin xyz="0 0 0" rpy="0 0 0" />
       <geometry>
-        <mesh filename="package://rm_description/meshes/glb/eco62/base_link.glb" />
+        <mesh filename="package://rm_description/meshes/dae/eco62/base_link.dae" />
       </geometry>
     </visual>
@@ -41,5 +41,5 @@
       <origin xyz="0 0 0" rpy="0 0 0" />
       <geometry>
-        <mesh filename="package://rm_description/meshes/glb/eco62/link_1.glb" />
+        <mesh filename="package://rm_description/meshes/dae/eco62/link_1.dae" />
       </geometry>
     </visual>
@@ -67,5 +67,5 @@
       <origin xyz="0 0 0" rpy="0 0 0" />
       <geometry>
-        <mesh filename="package://rm_description/meshes/glb/eco62/link_2.glb" />
+        <mesh filename="package://rm_description/meshes/dae/eco62/link_2.dae" />
       </geometry>
     </visual>
@@ -93,5 +93,5 @@
       <origin xyz="0 0 0" rpy="0 0 0" />
       <geometry>
-        <mesh filename="package://rm_description/meshes/glb/eco62/link_3.glb" />
+        <mesh filename="package://rm_description/meshes/dae/eco62/link_3.dae" />
       </geometry>
     </visual>
@@ -119,5 +119,5 @@
       <origin xyz="0 0 0" rpy="0 0 0" />
       <geometry>
-        <mesh filename="package://rm_description/meshes/glb/eco62/link_4.glb" />
+        <mesh filename="package://rm_description/meshes/dae/eco62/link_4.dae" />
       </geometry>
     </visual>
@@ -145,5 +145,5 @@
       <origin xyz="0 0 0" rpy="0 0 0" />
       <geometry>
-        <mesh filename="package://rm_description/meshes/glb/eco62/link_5.glb" />
+        <mesh filename="package://rm_description/meshes/dae/eco62/link_5.dae" />
       </geometry>
     </visual>
@@ -171,5 +171,5 @@
       <origin xyz="0 0 0" rpy="0 0 0" />
       <geometry>
-        <mesh filename="package://rm_description/meshes/glb/eco62/link_6.glb" />
+        <mesh filename="package://rm_description/meshes/dae/eco62/link_6.dae" />
       </geometry>
     </visual>

File: rm_description/urdf/imported/eco63_6fb.urdf.xacro (robot description, xacro)
@@ -22,5 +22,5 @@
       <origin xyz="0 0 0" rpy="0 0 0" />
       <geometry>
-        <mesh filename="package://rm_description/meshes/glb/base/base_v1.0.glb" />
+        <mesh filename="package://rm_description/meshes/dae/base/base_v1.0.dae" />
       </geometry>
     </visual>
@@ -41,5 +41,5 @@
       <origin xyz="0 0 0" rpy="0 0 0" />
       <geometry>
-        <mesh filename="package://rm_description/meshes/glb/eco63/link1_v1.0.glb" />
+        <mesh filename="package://rm_description/meshes/dae/eco63/link1_v1.0.dae" />
       </geometry>
     </visual>
@@ -67,5 +67,5 @@
       <origin xyz="0 0 0" rpy="0 0 0" />
       <geometry>
-        <mesh filename="package://rm_description/meshes/glb/eco63/link2_v1.0.glb" />
+        <mesh filename="package://rm_description/meshes/dae/eco63/link2_v1.0.dae" />
       </geometry>
     </visual>
@@ -93,5 +93,5 @@
       <origin xyz="0 0 0" rpy="0 0 0" />
       <geometry>
-        <mesh filename="package://rm_description/meshes/glb/eco63/link3_v1.0.glb" />
+        <mesh filename="package://rm_description/meshes/dae/eco63/link3_v1.0.dae" />
       </geometry>
     </visual>
@@ -119,5 +119,5 @@
       <origin xyz="0 0 0" rpy="0 0 0" />
       <geometry>
-        <mesh filename="package://rm_description/meshes/glb/eco63/link4_v1.0.glb" />
+        <mesh filename="package://rm_description/meshes/dae/eco63/link4_v1.0.dae" />
       </geometry>
     </visual>
@@ -145,5 +145,5 @@
       <origin xyz="0 0 0" rpy="0 0 0" />
       <geometry>
-        <mesh filename="package://rm_description/meshes/glb/eco63/link5_v1.0.glb" />
+        <mesh filename="package://rm_description/meshes/dae/eco63/link5_v1.0.dae" />
       </geometry>
     </visual>
@@ -171,5 +171,5 @@
       <origin xyz="0 0 0" rpy="0 0 0" />
       <geometry>
-        <mesh filename="package://rm_description/meshes/glb/eco63/link6Fb_v1.0.glb" />
+        <mesh filename="package://rm_description/meshes/dae/eco63/link6Fb_v1.0.dae" />
       </geometry>
     </visual>

File: rm_description/urdf/imported/eco63_standard.urdf.xacro (robot description, xacro)
@@ -22,5 +22,5 @@
       <origin xyz="0 0 0" rpy="0 0 0" />
       <geometry>
-        <mesh filename="package://rm_description/meshes/glb/base/base_v1.0.glb" />
+        <mesh filename="package://rm_description/meshes/dae/base/base_v1.0.dae" />
       </geometry>
     </visual>
@@ -41,5 +41,5 @@
       <origin xyz="0 0 0" rpy="0 0 0" />
       <geometry>
-        <mesh filename="package://rm_description/meshes/glb/eco63/link1_v1.0.glb" />
+        <mesh filename="package://rm_description/meshes/dae/eco63/link1_v1.0.dae" />
       </geometry>
     </visual>
@@ -67,5 +67,5 @@
       <origin xyz="0 0 0" rpy="0 0 0" />
       <geometry>
-        <mesh filename="package://rm_description/meshes/glb/eco63/link2_v1.0.glb" />
+        <mesh filename="package://rm_description/meshes/dae/eco63/link2_v1.0.dae" />
       </geometry>
     </visual>
@@ -93,5 +93,5 @@
       <origin xyz="0 0 0" rpy="0 0 0" />
       <geometry>
-        <mesh filename="package://rm_description/meshes/glb/eco63/link3_v1.0.glb" />
+        <mesh filename="package://rm_description/meshes/dae/eco63/link3_v1.0.dae" />
       </geometry>
     </visual>
@@ -119,5 +119,5 @@
       <origin xyz="0 0 0" rpy="0 0 0" />
       <geometry>
-        <mesh filename="package://rm_description/meshes/glb/eco63/link4_v1.0.glb" />
+        <mesh filename="package://rm_description/meshes/dae/eco63/link4_v1.0.dae" />
       </geometry>
     </visual>
@@ -145,5 +145,5 @@
       <origin xyz="0 0 0" rpy="0 0 0" />
       <geometry>
-        <mesh filename="package://rm_description/meshes/glb/eco63/link5_v1.0.glb" />
+        <mesh filename="package://rm_description/meshes/dae/eco63/link5_v1.0.dae" />
       </geometry>
     </visual>
@@ -171,5 +171,5 @@
       <origin xyz="0 0 0" rpy="0 0 0" />
       <geometry>
-        <mesh filename="package://rm_description/meshes/glb/eco63/link6_v1.0.glb" />
+        <mesh filename="package://rm_description/meshes/dae/eco63/link6_v1.0.dae" />
       </geometry>
     </visual>

File: rm_description/urdf/imported/eco65_6f.urdf.xacro (robot description, xacro)
@@ -16,5 +16,5 @@
       <origin xyz="0 0 0" rpy="0 0 0" />
       <geometry>
-        <mesh filename="package://rm_description/meshes/glb/base/base_v1.0.glb" />
+        <mesh filename="package://rm_description/meshes/dae/base/base_v1.0.dae" />
       </geometry>
     </visual>
@@ -35,5 +35,5 @@
       <origin xyz="0 0 0" rpy="0 0 0" />
       <geometry>
-        <mesh filename="package://rm_description/meshes/glb/eco65/link_1.glb" />
+        <mesh filename="package://rm_description/meshes/dae/eco65/link_1.dae" />
       </geometry>
     </visual>
@@ -61,5 +61,5 @@
       <origin xyz="0 0 0" rpy="0 0 0" />
       <geometry>
-        <mesh filename="package://rm_description/meshes/glb/eco65/link_2.glb" />
+        <mesh filename="package://rm_description/meshes/dae/eco65/link_2.dae" />
       </geometry>
     </visual>
@@ -87,5 +87,5 @@
       <origin xyz="0 0 0" rpy="0 0 0" />
       <geometry>
-        <mesh filename="package://rm_description/meshes/glb/eco65/link_3.glb" />
+        <mesh filename="package://rm_description/meshes/dae/eco65/link_3.dae" />
       </geometry>
     </visual>
@@ -113,5 +113,5 @@
       <origin xyz="0 0 0" rpy="0 0 0" />
       <geometry>
-        <mesh filename="package://rm_description/meshes/glb/eco65/link_4.glb" />
+        <mesh filename="package://rm_description/meshes/dae/eco65/link_4.dae" />
       </geometry>
     </visual>
@@ -139,5 +139,5 @@
       <origin xyz="0 0 0" rpy="0 0 0" />
       <geometry>
-        <mesh filename="package://rm_description/meshes/glb/eco65/link_5.glb" />
+        <mesh filename="package://rm_description/meshes/dae/eco65/link_5.dae" />
       </geometry>
     </visual>
@@ -165,5 +165,5 @@
       <origin xyz="0 0 0" rpy="0 0 0" />
       <geometry>
-        <mesh filename="package://rm_description/meshes/glb/eco65/link6_6fi.glb" />
+        <mesh filename="package://rm_description/meshes/dae/eco65/link6_6fi.dae" />
       </geometry>
     </visual>
