Commit message: feat: 改用 DAE 模型并适配 RViz2 和 Gazebo

File: rm_description/urdf/imported/eco65_6fb.urdf.xacro (robot description, xacro)
@@ -16,5 +16,5 @@
       <origin xyz="0 0 0" rpy="0 0 0" />
       <geometry>
-        <mesh filename="package://rm_description/meshes/glb/base/base_v1.0.glb" />
+        <mesh filename="package://rm_description/meshes/dae/base/base_v1.0.dae" />
       </geometry>
     </visual>
@@ -35,5 +35,5 @@
       <origin xyz="0 0 0" rpy="0 0 0" />
       <geometry>
-        <mesh filename="package://rm_description/meshes/glb/eco65/link_1.glb" />
+        <mesh filename="package://rm_description/meshes/dae/eco65/link_1.dae" />
       </geometry>
     </visual>
@@ -61,5 +61,5 @@
       <origin xyz="0 0 0" rpy="0 0 0" />
       <geometry>
-        <mesh filename="package://rm_description/meshes/glb/eco65/link_2.glb" />
+        <mesh filename="package://rm_description/meshes/dae/eco65/link_2.dae" />
       </geometry>
     </visual>
@@ -87,5 +87,5 @@
       <origin xyz="0 0 0" rpy="0 0 0" />
       <geometry>
-        <mesh filename="package://rm_description/meshes/glb/eco65/link_3.glb" />
+        <mesh filename="package://rm_description/meshes/dae/eco65/link_3.dae" />
       </geometry>
     </visual>
@@ -113,5 +113,5 @@
       <origin xyz="0 0 0" rpy="0 0 0" />
       <geometry>
-        <mesh filename="package://rm_description/meshes/glb/eco65/link_4.glb" />
+        <mesh filename="package://rm_description/meshes/dae/eco65/link_4.dae" />
       </geometry>
     </visual>
@@ -139,5 +139,5 @@
       <origin xyz="0 0 0" rpy="0 0 0" />
       <geometry>
-        <mesh filename="package://rm_description/meshes/glb/eco65/link_5.glb" />
+        <mesh filename="package://rm_description/meshes/dae/eco65/link_5.dae" />
       </geometry>
     </visual>
@@ -165,5 +165,5 @@
       <origin xyz="0 0 0" rpy="0 0 0" />
       <geometry>
-        <mesh filename="package://rm_description/meshes/glb/eco65/link_6_fb.glb" />
+        <mesh filename="package://rm_description/meshes/dae/eco65/link_6_fb.dae" />
       </geometry>
     </visual>

File: rm_description/urdf/imported/eco65_standard.urdf.xacro (robot description, xacro)
@@ -16,5 +16,5 @@
       <origin xyz="0 0 0" rpy="0 0 0" />
       <geometry>
-        <mesh filename="package://rm_description/meshes/glb/base/base_v1.0.glb" />
+        <mesh filename="package://rm_description/meshes/dae/base/base_v1.0.dae" />
       </geometry>
     </visual>
@@ -35,5 +35,5 @@
       <origin xyz="0 0 0" rpy="0 0 0" />
       <geometry>
-        <mesh filename="package://rm_description/meshes/glb/eco65/link_1.glb" />
+        <mesh filename="package://rm_description/meshes/dae/eco65/link_1.dae" />
       </geometry>
     </visual>
@@ -61,5 +61,5 @@
       <origin xyz="0 0 0" rpy="0 0 0" />
       <geometry>
-        <mesh filename="package://rm_description/meshes/glb/eco65/link_2.glb" />
+        <mesh filename="package://rm_description/meshes/dae/eco65/link_2.dae" />
       </geometry>
     </visual>
@@ -87,5 +87,5 @@
       <origin xyz="0 0 0" rpy="0 0 0" />
       <geometry>
-        <mesh filename="package://rm_description/meshes/glb/eco65/link_3.glb" />
+        <mesh filename="package://rm_description/meshes/dae/eco65/link_3.dae" />
       </geometry>
     </visual>
@@ -113,5 +113,5 @@
       <origin xyz="0 0 0" rpy="0 0 0" />
       <geometry>
-        <mesh filename="package://rm_description/meshes/glb/eco65/link_4.glb" />
+        <mesh filename="package://rm_description/meshes/dae/eco65/link_4.dae" />
       </geometry>
     </visual>
@@ -139,5 +139,5 @@
       <origin xyz="0 0 0" rpy="0 0 0" />
       <geometry>
-        <mesh filename="package://rm_description/meshes/glb/eco65/link_5.glb" />
+        <mesh filename="package://rm_description/meshes/dae/eco65/link_5.dae" />
       </geometry>
     </visual>
@@ -165,5 +165,5 @@
       <origin xyz="0 0 0" rpy="0 0 -1.57079632679" />
       <geometry>
-        <mesh filename="package://rm_description/meshes/glb/eco65/link_6.glb" />
+        <mesh filename="package://rm_description/meshes/dae/eco65/link_6.dae" />
       </geometry>
     </visual>

File: rm_description/urdf/imported/rx75_6fb.urdf.xacro (robot description, xacro)
@@ -31,5 +31,5 @@
       <origin xyz="0 0 0" rpy="0 0 0" />
       <geometry>
-        <mesh filename="package://rm_description/meshes/glb/rxl75/base_link.glb" />
+        <mesh filename="package://rm_description/meshes/dae/rxl75/base_link.dae" />
       </geometry>
     </visual>
@@ -50,5 +50,5 @@
       <origin xyz="0 0 0" rpy="0 0 0" />
       <geometry>
-        <mesh filename="package://rm_description/meshes/glb/rxl75/Link1.glb" />
+        <mesh filename="package://rm_description/meshes/dae/rxl75/Link1.dae" />
       </geometry>
     </visual>
@@ -76,5 +76,5 @@
       <origin xyz="0 0 0" rpy="0 0 0" />
       <geometry>
-        <mesh filename="package://rm_description/meshes/glb/rxl75/Link2.glb" />
+        <mesh filename="package://rm_description/meshes/dae/rxl75/Link2.dae" />
       </geometry>
     </visual>
@@ -102,5 +102,5 @@
       <origin xyz="0 0 0" rpy="0 0 0" />
       <geometry>
-        <mesh filename="package://rm_description/meshes/glb/rxl75/Link3.glb" />
+        <mesh filename="package://rm_description/meshes/dae/rxl75/Link3.dae" />
       </geometry>
     </visual>
@@ -128,5 +128,5 @@
       <origin xyz="0 0 0" rpy="0 0 0" />
       <geometry>
-        <mesh filename="package://rm_description/meshes/glb/rxl75/Link4.glb" />
+        <mesh filename="package://rm_description/meshes/dae/rxl75/Link4.dae" />
       </geometry>
     </visual>
@@ -154,5 +154,5 @@
       <origin xyz="0 0 0" rpy="0 0 0" />
       <geometry>
-        <mesh filename="package://rm_description/meshes/glb/rxl75/Link5.glb" />
+        <mesh filename="package://rm_description/meshes/dae/rxl75/Link5.dae" />
       </geometry>
     </visual>
@@ -180,5 +180,5 @@
       <origin xyz="0 0 0" rpy="0 0 0" />
       <geometry>
-        <mesh filename="package://rm_description/meshes/glb/rxl75/Link6.glb" />
+        <mesh filename="package://rm_description/meshes/dae/rxl75/Link6.dae" />
       </geometry>
     </visual>
@@ -212,5 +212,5 @@
       <origin xyz="0 0 0" rpy="0 0 0" />
       <geometry>
-        <mesh filename="package://rm_description/meshes/glb/rxl75/Link7-6FB.glb" />
+        <mesh filename="package://rm_description/meshes/dae/rxl75/Link7-6FB.dae" />
       </geometry>
     </visual>
@@ -227,5 +227,5 @@
       <origin xyz="0 0 0" rpy="0 0 0" />
       <geometry>
-        <mesh filename="package://rm_description/meshes/glb/rxl75/Link8.glb" />
+        <mesh filename="package://rm_description/meshes/dae/rxl75/Link8.dae" />
       </geometry>
     </visual>
@@ -251,5 +251,5 @@
       <origin xyz="0 0 0" rpy="0 0 0" />
       <geometry>
-        <mesh filename="package://rm_description/meshes/glb/rxr75/base_link.glb" />
+        <mesh filename="package://rm_description/meshes/dae/rxr75/base_link.dae" />
       </geometry>
     </visual>
@@ -270,5 +270,5 @@
       <origin xyz="0 0 0" rpy="0 0 0" />
       <geometry>
-        <mesh filename="package://rm_description/meshes/glb/rxr75/Link1.glb" />
+        <mesh filename="package://rm_description/meshes/dae/rxr75/Link1.dae" />
       </geometry>
     </visual>
@@ -296,5 +296,5 @@
       <origin xyz="0 0 0" rpy="0 0 0" />
       <geometry>
-        <mesh filename="package://rm_description/meshes/glb/rxr75/Link2.glb" />
+        <mesh filename="package://rm_description/meshes/dae/rxr75/Link2.dae" />
       </geometry>
     </visual>
@@ -322,5 +322,5 @@
       <origin xyz="0 0 0" rpy="0 0 0" />
       <geometry>
-        <mesh filename="package://rm_description/meshes/glb/rxr75/Link3.glb" />
+        <mesh filename="package://rm_description/meshes/dae/rxr75/Link3.dae" />
       </geometry>
     </visual>
@@ -348,5 +348,5 @@
       <origin xyz="0 0 0" rpy="0 0 0" />
       <geometry>
-        <mesh filename="package://rm_description/meshes/glb/rxr75/Link4.glb" />
+        <mesh filename="package://rm_description/meshes/dae/rxr75/Link4.dae" />
       </geometry>
     </visual>
@@ -374,5 +374,5 @@
       <origin xyz="0 0 0" rpy="0 0 0" />
       <geometry>
-        <mesh filename="package://rm_description/meshes/glb/rxr75/Link5.glb" />
+        <mesh filename="package://rm_description/meshes/dae/rxr75/Link5.dae" />
       </geometry>
     </visual>
@@ -400,5 +400,5 @@
       <origin xyz="0 0 0" rpy="0 0 0" />
       <geometry>
-        <mesh filename="package://rm_description/meshes/glb/rxr75/Link6.glb" />
+        <mesh filename="package://rm_description/meshes/dae/rxr75/Link6.dae" />
       </geometry>
     </visual>
@@ -432,5 +432,5 @@
       <origin xyz="0 0 0" rpy="0 0 0" />
       <geometry>
-        <mesh filename="package://rm_description/meshes/glb/rxr75/Link7-6FB.glb" />
+        <mesh filename="package://rm_description/meshes/dae/rxr75/Link7-6FB.dae" />
       </geometry>
     </visual>
@@ -447,5 +447,5 @@
       <origin xyz="0 0 0" rpy="0 0 0" />
       <geometry>
-        <mesh filename="package://rm_description/meshes/glb/rxr75/Link8.glb" />
+        <mesh filename="package://rm_description/meshes/dae/rxr75/Link8.dae" />
       </geometry>
     </visual>

File: rm_description/urdf/imported/rx75_6fb_v.urdf.xacro (robot description, xacro)
@@ -31,5 +31,5 @@
       <origin xyz="0 0 0" rpy="0 0 0" />
       <geometry>
-        <mesh filename="package://rm_description/meshes/glb/rxl75/base_link.glb" />
+        <mesh filename="package://rm_description/meshes/dae/rxl75/base_link.dae" />
       </geometry>
     </visual>
@@ -50,5 +50,5 @@
       <origin xyz="0 0 0" rpy="0 0 0" />
       <geometry>
-        <mesh filename="package://rm_description/meshes/glb/rxl75/Link1.glb" />
+        <mesh filename="package://rm_description/meshes/dae/rxl75/Link1.dae" />
       </geometry>
     </visual>
@@ -76,5 +76,5 @@
       <origin xyz="0 0 0" rpy="0 0 0" />
       <geometry>
-        <mesh filename="package://rm_description/meshes/glb/rxl75/Link2.glb" />
+        <mesh filename="package://rm_description/meshes/dae/rxl75/Link2.dae" />
       </geometry>
     </visual>
@@ -102,5 +102,5 @@
       <origin xyz="0 0 0" rpy="0 0 0" />
       <geometry>
-        <mesh filename="package://rm_description/meshes/glb/rxl75/Link3.glb" />
+        <mesh filename="package://rm_description/meshes/dae/rxl75/Link3.dae" />
       </geometry>
     </visual>
@@ -128,5 +128,5 @@
       <origin xyz="0 0 0" rpy="0 0 0" />
       <geometry>
-        <mesh filename="package://rm_description/meshes/glb/rxl75/Link4.glb" />
+        <mesh filename="package://rm_description/meshes/dae/rxl75/Link4.dae" />
       </geometry>
     </visual>
@@ -154,5 +154,5 @@
       <origin xyz="0 0 0" rpy="0 0 0" />
       <geometry>
-        <mesh filename="package://rm_description/meshes/glb/rxl75/Link5.glb" />
+        <mesh filename="package://rm_description/meshes/dae/rxl75/Link5.dae" />
       </geometry>
     </visual>
@@ -180,5 +180,5 @@
       <origin xyz="0 0 0" rpy="0 0 0" />
       <geometry>
-        <mesh filename="package://rm_description/meshes/glb/rxl75/Link6.glb" />
+        <mesh filename="package://rm_description/meshes/dae/rxl75/Link6.dae" />
       </geometry>
     </visual>
@@ -212,5 +212,5 @@
       <origin xyz="0 0 0" rpy="0 0 0" />
       <geometry>
-        <mesh filename="package://rm_description/meshes/glb/rxl75/Link7-6FB-V.glb" />
+        <mesh filename="package://rm_description/meshes/dae/rxl75/Link7-6FB-V.dae" />
       </geometry>
     </visual>
@@ -227,5 +227,5 @@
       <origin xyz="0 0 0" rpy="0 0 0" />
       <geometry>
-        <mesh filename="package://rm_description/meshes/glb/rxl75/Link8.glb" />
+        <mesh filename="package://rm_description/meshes/dae/rxl75/Link8.dae" />
       </geometry>
     </visual>
@@ -251,5 +251,5 @@
       <origin xyz="0 0 0" rpy="0 0 0" />
       <geometry>
-        <mesh filename="package://rm_description/meshes/glb/rxr75/base_link.glb" />
+        <mesh filename="package://rm_description/meshes/dae/rxr75/base_link.dae" />
       </geometry>
     </visual>
@@ -270,5 +270,5 @@
       <origin xyz="0 0 0" rpy="0 0 0" />
       <geometry>
-        <mesh filename="package://rm_description/meshes/glb/rxr75/Link1.glb" />
+        <mesh filename="package://rm_description/meshes/dae/rxr75/Link1.dae" />
       </geometry>
     </visual>
@@ -296,5 +296,5 @@
       <origin xyz="0 0 0" rpy="0 0 0" />
       <geometry>
-        <mesh filename="package://rm_description/meshes/glb/rxr75/Link2.glb" />
+        <mesh filename="package://rm_description/meshes/dae/rxr75/Link2.dae" />
       </geometry>
     </visual>
@@ -322,5 +322,5 @@
       <origin xyz="0 0 0" rpy="0 0 0" />
       <geometry>
-        <mesh filename="package://rm_description/meshes/glb/rxr75/Link3.glb" />
+        <mesh filename="package://rm_description/meshes/dae/rxr75/Link3.dae" />
       </geometry>
     </visual>
@@ -348,5 +348,5 @@
       <origin xyz="0 0 0" rpy="0 0 0" />
       <geometry>
-        <mesh filename="package://rm_description/meshes/glb/rxr75/Link4.glb" />
+        <mesh filename="package://rm_description/meshes/dae/rxr75/Link4.dae" />
       </geometry>
     </visual>
@@ -374,5 +374,5 @@
       <origin xyz="0 0 0" rpy="0 0 0" />
       <geometry>
-        <mesh filename="package://rm_description/meshes/glb/rxr75/Link5.glb" />
+        <mesh filename="package://rm_description/meshes/dae/rxr75/Link5.dae" />
       </geometry>
     </visual>
@@ -400,5 +400,5 @@
       <origin xyz="0 0 0" rpy="0 0 0" />
       <geometry>
-        <mesh filename="package://rm_description/meshes/glb/rxr75/Link6.glb" />
+        <mesh filename="package://rm_description/meshes/dae/rxr75/Link6.dae" />
       </geometry>
     </visual>
@@ -432,5 +432,5 @@
       <origin xyz="0 0 0" rpy="0 0 0" />
       <geometry>
-        <mesh filename="package://rm_description/meshes/glb/rxr75/Link7-6FB-V.glb" />
+        <mesh filename="package://rm_description/meshes/dae/rxr75/Link7-6FB-V.dae" />
       </geometry>
     </visual>
@@ -447,5 +447,5 @@
       <origin xyz="0 0 0" rpy="0 0 0" />
       <geometry>
-        <mesh filename="package://rm_description/meshes/glb/rxr75/Link8.glb" />
+        <mesh filename="package://rm_description/meshes/dae/rxr75/Link8.dae" />
       </geometry>
     </visual>
